Commit message: Added Sonars!

File: gazebo_naoqi_control/models/nao.urdf (robot description, URDF)
Before this commit: robot naoH25V40, 76 links, 75 joints
Links:
- removed link ImuAccelerometer_frame
- removed link ImuGyrometer_frame
- removed link imu
- added link CameraBottom_optical_frame
- added link CameraTop_optical_frame
- added link ImuTorsoAccelerometer_frame
- added link ImuTorsoGyrometer_frame
- added link LAnklePitch_link, mass 0.13416; collision mesh filename=package://nao_meshes/meshes/V40/LAnklePitch_0.10.stl scale=0.1 0.1 0.1; visual mesh filename=package://nao_meshes/meshes/V40/LAnklePitch.dae scale=0.1 0.1 0.1
- added link MicroFrontCenter_frame
- added link MicroRearCenter_frame
- added link MicroSurroundLeft_frame
- added link MicroSurroundRight_frame
- added link RAnklePitch_link, mass 0.13416; collision mesh filename=package://nao_meshes/meshes/V40/RAnklePitch_0.10.stl scale=0.1 0.1 0.1; visual mesh filename=package://nao_meshes/meshes/V40/RAnklePitch.dae scale=0.1 0.1 0.1
- link LFinger11_link: mass 0.2e-5 -> 2e-06
- link LFinger12_link: mass 0.2e-5 -> 2e-06
- link LFinger13_link: mass 0.2e-5 -> 2e-06
- link LFinger21_link: mass 0.2e-5 -> 2e-06
- link LFinger22_link: mass 0.2e-5 -> 2e-06
- link LFinger23_link: mass 0.2e-5 -> 2e-06
- link LThumb1_link: mass 0.2e-5 -> 2e-06
- link LThumb2_link: mass 0.2e-5 -> 2e-06
- link RFinger11_link: mass 0.2e-5 -> 2e-06
- link RFinger12_link: mass 0.2e-5 -> 2e-06
- link RFinger13_link: mass 0.2e-5 -> 2e-06
- link RFinger21_link: mass 0.2e-5 -> 2e-06
- link RFinger22_link: mass 0.2e-5 -> 2e-06
- link RFinger23_link: mass 0.2e-5 -> 2e-06
- link RThumb1_link: mass 0.2e-5 -> 2e-06
- link RThumb2_link: mass 0.2e-5 -> 2e-06
- link l_ankle: mass 0.13416 -> 0.16184; geometry collision mesh filename=package://nao_meshes/meshes/V40/LAnkleRoll_0.10.stl scale=0.1 0.1 0.1; visual mesh filename=package://nao_meshes/meshes/V40/LAnkleRoll.dae scale=0.1 0.1 0.1
- link l_sole: mass 0.16184 -> None; geometry 
- link r_ankle: mass 0.13416 -> 0.16184; geometry collision mesh filename=package://nao_meshes/meshes/V40/RAnkleRoll_0.10.stl scale=0.1 0.1 0.1; visual mesh filename=package://nao_meshes/meshes/V40/RAnkleRoll.dae scale=0.1 0.1 0.1
- link r_sole: mass 0.16184 -> None; geometry 
Joints:
- removed joint CameraBottom_joint
- removed joint CameraTop_joint
- removed joint ChestButton_joint
- removed joint HeadTouchFront_joint
- removed joint HeadTouchMiddle_joint
- removed joint HeadTouchRear_joint
- removed joint ImuAccelerometer_joint
- removed joint ImuGyrometer_joint
- removed joint LFinger1
- removed joint LFinger2
- removed joint LFootBumperLeft_joint
- removed joint LFootBumperRight_joint
- removed joint LFsrFL_joint
- removed joint LFsrFR_joint
- removed joint LFsrRL_joint
- removed joint LFsrRR_joint
- removed joint LHandTouchBack_joint
- removed joint LHandTouchLeft_joint
- removed joint LHandTouchRight_joint
- removed joint LInfraRed_joint
- removed joint LSonar_joint
- removed joint LThumb12
- removed joint RFinger1
- removed joint RFinger2
- removed joint RFootBumperLeft_joint
- removed joint RFootBumperRight_joint
- removed joint RFsrFL_joint
- removed joint RFsrFR_joint
- removed joint RFsrRL_joint
- removed joint RFsrRR_joint
- removed joint RHandTouchBack_joint
- removed joint RHandTouchLeft_joint
- removed joint RHandTouchRight_joint
- removed joint RInfraRed_joint
- removed joint RSonar_joint
- removed joint RThumb12
- removed joint base_joint
- removed joint torso-imu
- added joint Accelerometer_sensor_fixedjoint: type fixed, parent torso, child ImuTorsoAccelerometer_frame, origin xyz=-0.008 0.00606 0.027 rpy=0 0 0, axis 0 0 0
- added joint CameraBottom_optical_frame_joint: type fixed, parent CameraBottom_frame, child CameraBottom_optical_frame, origin xyz=0 0 0 rpy=-1.57079632679 0 -1.57079632679
- added joint CameraBottom_sensor_fixedjoint: type fixed, parent Head, child CameraBottom_frame, origin xyz=0.05071 0 0.01774 rpy=0 0.692896 0, axis 0 0 0
- added joint CameraTop_optical_frame_joint: type fixed, parent CameraTop_frame, child CameraTop_optical_frame, origin xyz=0 0 0 rpy=-1.57079632679 0 -1.57079632679
- added joint CameraTop_sensor_fixedjoint: type fixed, parent Head, child CameraTop_frame, origin xyz=0.05871 0 0.06364 rpy=0 0.0209435 0, axis 0 0 0
- added joint ChestBoard/Button_sensor_fixedjoint: type fixed, parent torso, child ChestButton_frame, origin xyz=0.049871 0.001588 0.055163 rpy=0 0 0, axis 0 0 0
- added joint Gyrometer_sensor_fixedjoint: type fixed, parent torso, child ImuTorsoGyrometer_frame, origin xyz=-0.008 0.006 0.029 rpy=0 0 0, axis 0 0 0
- added joint Head/Touch/Front_sensor_fixedjoint: type fixed, parent Head, child HeadTouchFront_frame, origin xyz=0.0312 0 0.1014 rpy=0 -1.1861 0, axis 0 0 0
- added joint Head/Touch/Middle_sensor_fixedjoint: type fixed, parent Head, child HeadTouchMiddle_frame, origin xyz=0.001 0 0.1099 rpy=3.14159 -1.57079 -3.14159, axis 0 0 0
- added joint Head/Touch/Rear_sensor_fixedjoint: type fixed, parent Head, child HeadTouchRear_frame, origin xyz=-0.0257 0 0.1045 rpy=3.14159 -1.33319 -3.14159, axis 0 0 0
- added joint InfraredL_sensor_fixedjoint: type fixed, parent Head, child LInfraRed_frame, origin xyz=0.0441 0.0257 0.0466 rpy=0 0 0, axis 0 0 0
- added joint InfraredR_sensor_fixedjoint: type fixed, parent Head, child RInfraRed_frame, origin xyz=0.0441 -0.0257 0.0466 rpy=0 0 0, axis 0 0 0
- added joint LFinger13: type continuous, parent LFinger12_link, child LFinger13_link, origin xyz=0.01436 0 0 rpy=0 0 -0.999899, axis 0 0 1.0, mimic joint=LHand multiplier=0.999899 offset=0
- added joint LFinger23: type continuous, parent LFinger22_link, child LFinger23_link, origin xyz=0.01436 0 0 rpy=0 0 -0.999899, axis 0 0 1.0, mimic joint=LHand multiplier=0.999899 offset=0
- added joint LFoot/Bumper/Left_sensor_fixedjoint: type fixed, parent l_ankle, child LFootBumperLeft_frame, origin xyz=0.0876 0.019 -0.0353 rpy=0 0 0, axis 0 0 0
- added joint LFoot/Bumper/Right_sensor_fixedjoint: type fixed, parent l_ankle, child LFootBumperRight_frame, origin xyz=0.0876 -0.014 -0.0353 rpy=0 0 0, axis 0 0 0
- added joint LFoot/FSR/FrontLeft_sensor_fixedjoint: type fixed, parent l_ankle, child LFsrFL_frame, origin xyz=0.07025 0.0299 -0.04511 rpy=0 0 0, axis 0 0 0
- added joint LFoot/FSR/FrontRight_sensor_fixedjoint: type fixed, parent l_ankle, child LFsrFR_frame, origin xyz=0.07025 -0.0231 -0.04511 rpy=0 0 0, axis 0 0 0
- added joint LFoot/FSR/RearLeft_sensor_fixedjoint: type fixed, parent l_ankle, child LFsrRL_frame, origin xyz=-0.03025 0.0299 -0.04511 rpy=0 0 0, axis 0 0 0
- added joint LFoot/FSR/RearRight_sensor_fixedjoint: type fixed, parent l_ankle, child LFsrRR_frame, origin xyz=-0.02965 -0.0191 -0.04511 rpy=0 0 0, axis 0 0 0
- added joint LHand/Touch/Back_sensor_fixedjoint: type fixed, parent l_wrist, child LHandTouchBack_frame, origin xyz=0.038 0 0.025 rpy=3.14159 -1.5708 3.14159, axis 0 0 0
- added joint LHand/Touch/Left_sensor_fixedjoint: type fixed, parent l_wrist, child LHandTouchLeft_frame, origin xyz=0.032 0.025 0.003 rpy=0 0 1.5708, axis 0 0 0
- added joint LHand/Touch/Right_sensor_fixedjoint: type fixed, parent l_wrist, child LHandTouchRight_frame, origin xyz=0.035 -0.025 0.0035 rpy=0 0 -1.5708, axis 0 0 0
- added joint LLeg_effector_fixedjoint: type fixed, parent l_ankle, child l_sole, origin xyz=0 0 -0.04511 rpy=0 0 0, axis 0 0 0
- added joint LThumb2: type continuous, parent LThumb1_link, child LThumb2_link, origin xyz=0.01436 0 0 rpy=0 0 -0.999899, axis 0 0 1.0, mimic joint=LHand multiplier=0.999899 offset=0
- added joint MicroFront_sensor_fixedjoint: type fixed, parent Head, child MicroFrontCenter_frame, origin xyz=0.041 0 0.091 rpy=0 0 0, axis 0 0 0
- added joint MicroLeft_sensor_fixedjoint: type fixed, parent Head, child MicroSurroundLeft_frame, origin xyz=-0.0195 0.0606 0.0331 rpy=0 0 0, axis 0 0 0
- added joint MicroRear_sensor_fixedjoint: type fixed, parent Head, child MicroRearCenter_frame, origin xyz=-0.0577 0 0.0693 rpy=0 0 0, axis 0 0 0
- added joint MicroRight_sensor_fixedjoint: type fixed, parent Head, child MicroSurroundRight_frame, origin xyz=-0.0195 -0.0606 0.0331 rpy=0 0 0, axis 0 0 0
- added joint RFinger13: type continuous, parent RFinger12_link, child RFinger13_link, origin xyz=0.01436 0 0 rpy=0 0 -0.999899, axis 0 0 1.0, mimic joint=RHand multiplier=0.999899 offset=0
- added joint RFinger23: type continuous, parent RFinger22_link, child RFinger23_link, origin xyz=0.01436 0 0 rpy=0 0 -0.999899, axis 0 0 1.0, mimic joint=RHand multiplier=0.999899 offset=0
- added joint RFoot/Bumper/Left_sensor_fixedjoint: type fixed, parent r_ankle, child RFootBumperLeft_frame, origin xyz=0.0876 0.014 -0.0353 rpy=0 0 0, axis 0 0 0
- added joint RFoot/Bumper/Right_sensor_fixedjoint: type fixed, parent r_ankle, child RFootBumperRight_frame, origin xyz=0.0876 -0.019 -0.0353 rpy=0 0 0, axis 0 0 0
- added joint RFoot/FSR/FrontLeft_sensor_fixedjoint: type fixed, parent r_ankle, child RFsrFL_frame, origin xyz=0.07025 0.0231 -0.04511 rpy=0 0 0, axis 0 0 0
- added joint RFoot/FSR/FrontRight_sensor_fixedjoint: type fixed, parent r_ankle, child RFsrFR_frame, origin xyz=0.07025 -0.0299 -0.04511 rpy=0 0 0, axis 0 0 0
- added joint RFoot/FSR/RearLeft_sensor_fixedjoint: type fixed, parent r_ankle, child RFsrRL_frame, origin xyz=-0.03025 0.0191 -0.04511 rpy=0 0 0, axis 0 0 0
- added joint RFoot/FSR/RearRight_sensor_fixedjoint: type fixed, parent r_ankle, child RFsrRR_frame, origin xyz=-0.02965 -0.0299 -0.04511 rpy=0 0 0, axis 0 0 0
- added joint RHand/Touch/Back_sensor_fixedjoint: type fixed, parent r_wrist, child RHandTouchBack_frame, origin xyz=0.038 0 0.025 rpy=3.14159 -1.5708 3.14159, axis 0 0 0
- added joint RHand/Touch/Left_sensor_fixedjoint: type fixed, parent r_wrist, child RHandTouchLeft_frame, origin xyz=0.032 0.025 0.003 rpy=0 0 1.5708, axis 0 0 0
- added joint RHand/Touch/Right_sensor_fixedjoint: type fixed, parent r_wrist, child RHandTouchRight_frame, origin xyz=0.035 -0.025 0.0035 rpy=0 0 -1.5708, axis 0 0 0
- added joint RLeg_effector_fixedjoint: type fixed, parent r_ankle, child r_sole, origin xyz=0 0 -0.04511 rpy=0 0 0, axis 0 0 0
- added joint RThumb2: type continuous, parent RThumb1_link, child RThumb2_link, origin xyz=0.01436 0 0 rpy=0 0 -0.999899, axis 0 0 1.0, mimic joint=RHand multiplier=0.999899 offset=0
- added joint Sonar/Left_sensor_fixedjoint: type fixed, parent torso, child LSonar_frame, origin xyz=0.00558253 0.0192068 0.0623853 rpy=-0.00478508 -1.52714663 0.392441, axis 0 0 0
- added joint Sonar/Right_sensor_fixedjoint: type fixed, parent torso, child RSonar_frame, origin xyz=0.00558253 -0.0192068 0.0623853 rpy=0.00478508 -1.52714663 -0.392441, axis 0 0 0
- added joint base_link_fixedjoint: type fixed, parent base_link, child torso, origin xyz=0 0 0 rpy=0 0 0, axis 0 0 0
- joint HeadPitch: limit lower=-0.671952 upper=0.514872 effort=1.2 velocity=7.19407 -> lower=-0.671952 upper=0.514872 effort=1.532 velocity=7.19407
- joint HeadYaw: limit lower=-2.08567 upper=2.08567 effort=1.2 velocity=8.26797 -> lower=-2.08567 upper=2.08567 effort=1.547 velocity=8.26797
- joint LAnklePitch: child l_ankle -> LAnklePitch_link; limit lower=-1.18944 upper=0.922581 effort=3.2 velocity=6.40239 -> lower=-1.18944 upper=0.922581 effort=3.023 velocity=6.40239
- joint LAnkleRoll: child l_sole -> l_ankle; limit lower=-0.397761 upper=0.768992 effort=3.2 velocity=4.16174 -> lower=-0.397761 upper=0.768992 effort=3.348 velocity=4.16174; parent l_ankle -> LAnklePitch_link
- joint LElbowRoll: limit lower=-1.54462 upper=-0.0349066 effort=1.2 velocity=7.19407 -> lower=-1.54462 upper=-0.0349066 effort=1.532 velocity=7.19407
- joint LElbowYaw: limit lower=-2.08567 upper=2.08567 effort=1.2 velocity=8.26797 -> lower=-2.08567 upper=2.08567 effort=1.547 velocity=8.26797
- joint LFinger11: axis 0 1 0 -> 0 0 1.0; child LFinger12_link -> LFinger11_link; limit lower=0.0 upper=0.785398163398 effort=10.0 velocity=3.0 -> (none); mimic joint=LHand multiplier=-0.785398163398 offset=0.785398163398 -> joint=LHand multiplier=0.999899 offset=0; origin xyz=0.01436 0 0 rpy=0 0 0 -> xyz=0.06907 0.01157 -0.00304 rpy=1.8862 0.976662 0.264067; parent LFinger11_link -> l_wrist; type revolute -> continuous
- joint LFinger12: axis 0 1 0 -> 0 0 1.0; child LFinger13_link -> LFinger12_link; limit lower=0.0 upper=0.785398163398 effort=10.0 velocity=3.0 -> (none); mimic joint=LHand multiplier=-0.785398163398 offset=0.785398163398 -> joint=LHand multiplier=0.999899 offset=0; origin xyz=0.01436 0 0 rpy=0 0 0 -> xyz=0.01436 0 0 rpy=0 0 -0.999899; parent LFinger12_link -> LFinger11_link; type revolute -> continuous
- joint LFinger21: axis 0 1 0 -> 0 0 1.0; child LFinger22_link -> LFinger21_link; limit lower=0.0 upper=0.785398163398 effort=10.0 velocity=3.0 -> (none); mimic joint=LHand multiplier=-0.785398163398 offset=0.785398163398 -> joint=LHand multiplier=0.999899 offset=0; origin xyz=0.01436 0 0 rpy=0 0 0 -> xyz=0.06907 -0.01157 -0.00304 rpy=1.25539 0.976662 -0.264067; parent LFinger21_link -> l_wrist; type revolute -> continuous
- joint LFinger22: axis 0 1 0 -> 0 0 1.0; child LFinger23_link -> LFinger22_link; limit lower=0.0 upper=0.785398163398 effort=10.0 velocity=3.0 -> (none); mimic joint=LHand multiplier=-0.785398163398 offset=0.785398163398 -> joint=LHand multiplier=0.999899 offset=0; origin xyz=0.01436 0 0 rpy=0 0 0 -> xyz=0.01436 0 0 rpy=0 0 -0.999899; parent LFinger22_link -> LFinger21_link; type revolute -> continuous
- joint LHand: axis (none) -> 1.0 0 0; limit lower=0 upper=1.0 effort=0.177576 velocity=3 -> lower=0 upper=1.0 effort=0.292 velocity=8.33
- joint LHipPitch: limit lower=-1.53589 upper=0.48398 effort=3.2 velocity=6.40239 -> lower=-1.53589 upper=0.48398 effort=3.023 velocity=6.40239
- joint LHipRoll: limit lower=-0.379435 upper=0.79046 effort=3.2 velocity=4.16174 -> lower=-0.379435 upper=0.79046 effort=3.348 velocity=4.16174
- joint LHipYawPitch: limit lower=-1.14529 upper=0.740718 effort=3.2 velocity=4.16174 -> lower=-1.14529 upper=0.740718 effort=3.348 velocity=4.16174
- joint LKneePitch: limit lower=-0.0923279 upper=2.11255 effort=3.2 velocity=6.40239 -> lower=-0.0923279 upper=2.11255 effort=3.023 velocity=6.40239
- joint LShoulderPitch: limit lower=-2.08567 upper=2.08567 effort=1.2 velocity=8.26797 -> lower=-2.08567 upper=2.08567 effort=1.329 velocity=8.26797
- joint LShoulderRoll: limit lower=-0.314159 upper=1.32645 effort=1.2 velocity=7.19407 -> lower=-0.314159 upper=1.32645 effort=1.7835 velocity=7.19407
- joint LThumb1: axis 0 1 0 -> 0 0 1.0; limit lower=0.0 upper=0.785398163398 effort=10.0 velocity=3.0 -> (none); mimic joint=LHand multiplier=-0.785398163398 offset=0.785398163398 -> joint=LHand multiplier=0.999899 offset=0; origin xyz=0.04895 0 -0.02638 rpy=3.14159265359 0.785398163398 0 -> xyz=0.04895 0 -0.02638 rpy=-1.5708 0.0472984 -3.26826e-08; type revolute -> continuous
- joint LWristYaw: limit lower=-1.82387 upper=1.82387 effort=0.76 velocity=24.6229 -> lower=-1.82387 upper=1.82387 effort=0.4075 velocity=24.6229
- joint RAnklePitch: child r_ankle -> RAnklePitch_link; limit lower=-1.1863 upper=0.932006 effort=3.2 velocity=6.40239 -> lower=-1.1863 upper=0.932006 effort=3.0226 velocity=6.40239
- joint RAnkleRoll: child r_sole -> r_ankle; limit lower=-0.768992 upper=0.397935 effort=3.2 velocity=4.16174 -> lower=-0.768992 upper=0.397761 effort=3.348 velocity=4.16174; parent r_ankle -> RAnklePitch_link
- joint RElbowRoll: limit lower=0.0349066 upper=1.54462 effort=1.2 velocity=7.19407 -> lower=0.0349066 upper=1.54462 effort=1.532 velocity=7.19407
- joint RElbowYaw: limit lower=-2.08567 upper=2.08567 effort=1.2 velocity=8.26797 -> lower=-2.08567 upper=2.08567 effort=1.547 velocity=8.26797
- joint RFinger11: axis 0 1 0 -> 0 0 1.0; child RFinger12_link -> RFinger11_link; limit lower=0.0 upper=0.785398163398 effort=10.0 velocity=3.0 -> (none); mimic joint=RHand multiplier=-0.785398163398 offset=0.785398163398 -> joint=RHand multiplier=0.999899 offset=0; origin xyz=0.01436 0 0 rpy=0 0 0 -> xyz=0.06907 0.01157 -0.00304 rpy=1.8862 0.976662 0.264067; parent RFinger11_link -> r_wrist; type revolute -> continuous
- joint RFinger12: axis 0 1 0 -> 0 0 1.0; child RFinger13_link -> RFinger12_link; limit lower=0.0 upper=0.785398163398 effort=10.0 velocity=3.0 -> (none); mimic joint=RHand multiplier=-0.785398163398 offset=0.785398163398 -> joint=RHand multiplier=0.999899 offset=0; origin xyz=0.01436 0 0 rpy=0 0 0 -> xyz=0.01436 0 0 rpy=0 0 -0.999899; parent RFinger12_link -> RFinger11_link; type revolute -> continuous
- joint RFinger21: axis 0 1 0 -> 0 0 1.0; child RFinger22_link -> RFinger21_link; limit lower=0.0 upper=0.785398163398 effort=10.0 velocity=3.0 -> (none); mimic joint=RHand multiplier=-0.785398163398 offset=0.785398163398 -> joint=RHand multiplier=0.999899 offset=0; origin xyz=0.01436 0 0 rpy=0 0 0 -> xyz=0.06907 -0.01157 -0.00304 rpy=1.25539 0.976662 -0.264067; parent RFinger21_link -> r_wrist; type revolute -> continuous
- joint RFinger22: axis 0 1 0 -> 0 0 1.0; child RFinger23_link -> RFinger22_link; limit lower=0.0 upper=0.785398163398 effort=10.0 velocity=3.0 -> (none); mimic joint=RHand multiplier=-0.785398163398 offset=0.785398163398 -> joint=RHand multiplier=0.999899 offset=0; origin xyz=0.01436 0 0 rpy=0 0 0 -> xyz=0.01436 0 0 rpy=0 0 -0.999899; parent RFinger22_link -> RFinger21_link; type revolute -> continuous
- joint RHand: axis (none) -> 1.0 0 0; limit lower=0 upper=1.0 effort=0.177576 velocity=3 -> lower=0 upper=1.0 effort=0.292 velocity=8.33; origin xyz=0.05775 0 -0.01231 rpy=0 0 0 -> xyz=0.05775 0 -0.01213 rpy=0 0 0
- joint RHipPitch: limit lower=-1.53589 upper=0.48398 effort=3.2 velocity=6.40239 -> lower=-1.53589 upper=0.48398 effort=3.0226 velocity=6.40239
- joint RHipRoll: limit lower=-0.79046 upper=0.379435 effort=3.2 velocity=4.16174 -> lower=-0.79046 upper=0.379435 effort=3.348 velocity=4.16174
- joint RHipYawPitch: limit lower=-1.14529 upper=0.740718 effort=3.2 velocity=4.16174 -> lower=-1.14529 upper=0.740718 effort=3.348 velocity=4.16174; mimic (none) -> joint=LHipYawPitch multiplier=1.0 offset=0
- joint RKneePitch: limit lower=-0.0923279 upper=2.11255 effort=3.2 velocity=6.40239 -> lower=-0.0923279 upper=2.11255 effort=3.0226 velocity=6.40239
- joint RShoulderPitch: limit lower=-2.08567 upper=2.08567 effort=1.2 velocity=8.26797 -> lower=-2.08567 upper=2.08567 effort=1.329 velocity=8.26797
- joint RShoulderRoll: limit lower=-1.32645 upper=0.314159 effort=1.2 velocity=7.19407 -> lower=-1.32645 upper=0.314159 effort=1.783 velocity=7.19407
- joint RThumb1: axis 0 1 0 -> 0 0 1.0; limit lower=0.0 upper=0.785398163398 effort=10.0 velocity=3.0 -> (none); mimic joint=RHand multiplier=-0.785398163398 offset=0.785398163398 -> joint=RHand multiplier=0.999899 offset=0; origin xyz=0.04895 0 -0.02638 rpy=3.14159265359 0.785398163398 0 -> xyz=0.04895 0 -0.02638 rpy=-1.5708 0.0472984 -3.26826e-08; type revolute -> continuous
- joint RWristYaw: limit lower=-1.82387 upper=1.82387 effort=0.76 velocity=24.6229 -> lower=-1.82387 upper=1.82387 effort=0.4075 velocity=24.6229
- joint gaze_joint: origin xyz=0.05871 0 0.06364 rpy=0 0.0209 0 -> xyz=0.05871 0 0.06364 rpy=0 0 0

Commit message: Added FSRs! Almost working..Everything but the gait!

File: gazebo_naoqi_control/models/nao.urdf (robot description, URDF)
Before this commit: robot naoH25V40, 83 links, 82 joints
Links:
- link LFsrFL_frame: mass None -> 0.2e-5; geometry collision box size=0.01 0.01 0.001
- link LFsrFR_frame: mass None -> 0.2e-5; geometry collision box size=0.01 0.01 0.001
- link LFsrRL_frame: mass None -> 0.2e-5; geometry collision box size=0.01 0.01 0.001
- link LFsrRR_frame: mass None -> 0.2e-5; geometry collision box size=0.01 0.01 0.001
- link RFsrFL_frame: mass None -> 0.2e-5; geometry collision box size=0.01 0.01 0.001
- link RFsrFR_frame: mass None -> 0.2e-5; geometry collision box size=0.01 0.01 0.001
- link RFsrRL_frame: mass None -> 0.2e-5; geometry collision box size=0.01 0.01 0.001
- link RFsrRR_frame: mass None -> 0.2e-5; geometry collision box size=0.01 0.01 0.001
Joints:
- joint LFoot/FSR/FrontLeft_sensor_fixedjoint: axis 0 0 0 -> 0 0 1; type fixed -> continuous
- joint LFoot/FSR/FrontRight_sensor_fixedjoint: axis 0 0 0 -> 0 0 1; type fixed -> continuous
- joint LFoot/FSR/RearLeft_sensor_fixedjoint: axis 0 0 0 -> 0 0 1; type fixed -> continuous
- joint LFoot/FSR/RearRight_sensor_fixedjoint: axis 0 0 0 -> 0 0 1; type fixed -> continuous
- joint RFoot/FSR/FrontLeft_sensor_fixedjoint: axis 0 0 0 -> 0 0 1; type fixed -> continuous
- joint RFoot/FSR/FrontRight_sensor_fixedjoint: axis 0 0 0 -> 0 0 1; type fixed -> continuous
- joint RFoot/FSR/RearLeft_sensor_fixedjoint: axis 0 0 0 -> 0 0 1; type fixed -> continuous
- joint RFoot/FSR/RearRight_sensor_fixedjoint: axis 0 0 0 -> 0 0 1; type fixed -> continuous
