Commit message: Small restructure in code/xacro for performance gain..Control period of 100Hz as default

File: gazebo_naoqi_control/models/model.xacro (robot description, xacro)
@@ -3,6 +3,6 @@
   <!-- Specify properties needed -->
   <xacro:property name="robotNamespace" value="/nao_dcm"/>
-  <!-- <xacro:property name="controlPeriod" value="0.001"/> -->
-  <xacro:property name="gazeboControlPeriod" value="true"/>
+  <xacro:property name="controlPeriod" value="0.01"/> <!-- 100Hz control -->
+  <xacro:property name="gazeboControlPeriod" value="false"/>
   <xacro:property name="port" value="9559"/>
   <xacro:property name="modelType" value="NAOH25V40"/>

Commit message: Sensors update only on their update rate! Improved performance..

File: gazebo_naoqi_control/models/model.xacro (robot description, xacro)
@@ -3,6 +3,6 @@
   <!-- Specify properties needed -->
   <xacro:property name="robotNamespace" value="/nao_dcm"/>
-  <xacro:property name="controlPeriod" value="0.01"/> <!-- 100Hz control -->
-  <xacro:property name="gazeboControlPeriod" value="false"/>
+  <!-- <xacro:property name="controlPeriod" value="0.01"/> --> <!-- 100Hz control -->
+  <xacro:property name="gazeboControlPeriod" value="true"/>
   <xacro:property name="port" value="9559"/>
   <xacro:property name="modelType" value="NAOH25V40"/>

File: gazebo_naoqi_control/models/nao.xacro (robot description, xacro)
@@ -1446,5 +1446,5 @@
       <origin xyz="0 0 0" rpy="0 0 0" />
       <geometry>
-        <box size="0.01 0.01 0.001" />
+        <box size="0.01 0.01 0.005" />
       </geometry>
     </collision>
@@ -1471,5 +1471,5 @@
       <origin xyz="0 0 0" rpy="0 0 0" />
       <geometry>
-        <box size="0.01 0.01 0.001" />
+        <box size="0.01 0.01 0.005" />
       </geometry>
     </collision>
@@ -1490,5 +1490,5 @@
       <origin xyz="0 0 0" rpy="0 0 0" />
       <geometry>
-        <box size="0.01 0.01 0.001" />
+        <box size="0.01 0.01 0.005" />
       </geometry>
     </collision>
@@ -1530,5 +1530,5 @@
       <origin xyz="0 0 0" rpy="0 0 0" />
       <geometry>
-        <box size="0.01 0.01 0.001" />
+        <box size="0.01 0.01 0.005" />
       </geometry>
     </collision>
@@ -1556,5 +1556,5 @@
       <origin xyz="0 0 0" rpy="0 0 0" />
       <geometry>
-        <box size="0.01 0.01 0.001" />
+        <box size="0.01 0.01 0.005" />
       </geometry>
     </collision>
@@ -1617,5 +1617,5 @@
       <origin xyz="0 0 0" rpy="0 0 0" />
       <geometry>
-        <box size="0.01 0.01 0.001" />
+        <box size="0.01 0.01 0.005" />
       </geometry>
     </collision>
@@ -1632,5 +1632,6 @@
     <child link="LSonar_frame"/>
     <!-- <origin rpy="-0.00478508 -1.52714663 0.392441" xyz="0.00558253 0.0192068 0.0623853"/> -->
-    <origin rpy="-0.00478508 0.0436497 0.392441" xyz="0.00558253 0.0192068 0.0623853"/>
+    <!-- <origin rpy="-0.00478508 0.0436497 0.392441" xyz="0.00558253 0.0192068 0.0623853"/> -->
+    <origin xyz="0.0477 0.0416 0.0509" rpy="0 0.2618 0.4363"/>
     <axis xyz="0 0 0"/>
   </joint>
@@ -1651,5 +1652,5 @@
       <origin xyz="0 0 0" rpy="0 0 0" />
       <geometry>
-        <box size="0.01 0.01 0.001" />
+        <box size="0.01 0.01 0.005" />
       </geometry>
     </collision>
@@ -1670,5 +1671,5 @@
       <origin xyz="0 0 0" rpy="0 0 0" />
       <geometry>
-        <box size="0.01 0.01 0.001" />
+        <box size="0.01 0.01 0.005" />
       </geometry>
     </collision>
@@ -1685,5 +1686,6 @@
     <child link="RSonar_frame"/>
     <!-- <origin rpy="0.00478508 -1.52714663 -0.392441" xyz="0.00558253 -0.0192068 0.0623853"/> -->
-    <origin rpy="0.00478508 0.0436497 -0.392441" xyz="0.00558253 -0.0192068 0.0623853"/>
+    <!-- <origin rpy="0.00478508 0.0436497 -0.392441" xyz="0.00558253 -0.0192068 0.0623853"/> -->
+    <origin xyz="0.0477 -0.0416 0.0509" rpy="0 0.2618 -0.4363"/>
     <axis xyz="0 0 0"/>
   </joint>
