Commit message: READY for publishing

File: gazebo_naoqi_control/models/nao.xacro (robot description, xacro)
@@ -7,10 +7,23 @@
  ****** File automatically generated by generate_urdf.py script ******
  *********************************************************************-->
-<robot name="naoH25V40" xmlns:xacro="http://www.ros.org/wiki/xacro">
+<robot xmlns:xacro="http://www.ros.org/wiki/xacro">
+  <!-- Xacro properties -->
+  <xacro:property name="robotNamespace" default="/nao_dcm"/>
+  <xacro:property name="controlPeriod" default="0.001"/>
+  <xacro:property name="gazeboControlPeriod" defalut="true"/>
+  <xacro:property name="port" default="9559"/>
+  <xacro:property name="modelType" default="NAOH25V40"/>
+  <!-- Gazebo NAOqi Plugin -->
   <gazebo>
     <plugin filename="libgazebo_naoqi_control.so" name="gazebo_naoqi_control">
-      <robotNamespace>/nao_dcm</robotNamespace>
+      <robotNamespace>${robotNamespace}</robotNamespace>
+      <xacro:unless value="${gazeboControlPeriod}">
+        <controlPeriod>${controlPeriod}</controlPeriod>
+      </xacro:unless>
+      <port>${port}</port>
+      <modelType>${modelType}</modelType>
     </plugin>
   </gazebo>
+  <!-- REST OF GAZEBO AND URDF -->
   <gazebo reference="torso">
     <mu1>0.5</mu1>
@@ -457,4 +470,11 @@
   </gazebo>
   <gazebo reference="RFsrRL_frame">
+    <mu1>0.5</mu1>
+    <mu2>0.5</mu2>
+    <selfCollide>false</selfCollide>
+    <turnGravityOff>false</turnGravityOff>
+    <fdir1>1 0 0</fdir1>
+    <maxVel>0.1</maxVel>
+    <minDepth>0.003</minDepth>
     <sensor name="RFoot/FSR/RearLeft" type="contact">
       <always_on>1</always_on>
@@ -468,4 +488,11 @@
   </gazebo>
   <gazebo reference="RFsrRR_frame">
+    <mu1>0.5</mu1>
+    <mu2>0.5</mu2>
+    <selfCollide>false</selfCollide>
+    <turnGravityOff>false</turnGravityOff>
+    <fdir1>1 0 0</fdir1>
+    <maxVel>0.1</maxVel>
+    <minDepth>0.003</minDepth>
     <sensor name="RFoot/FSR/RearRight" type="contact">
       <always_on>1</always_on>
@@ -479,4 +506,11 @@
   </gazebo>
   <gazebo reference="RFsrFL_frame">
+    <mu1>0.5</mu1>
+    <mu2>0.5</mu2>
+    <selfCollide>false</selfCollide>
+    <turnGravityOff>false</turnGravityOff>
+    <fdir1>1 0 0</fdir1>
+    <maxVel>0.1</maxVel>
+    <minDepth>0.003</minDepth>
     <sensor name="RFoot/FSR/FrontLeft" type="contact">
       <always_on>1</always_on>
@@ -490,4 +524,11 @@
   </gazebo>
   <gazebo reference="RFsrFR_frame">
+    <mu1>0.5</mu1>
+    <mu2>0.5</mu2>
+    <selfCollide>false</selfCollide>
+    <turnGravityOff>false</turnGravityOff>
+    <fdir1>1 0 0</fdir1>
+    <maxVel>0.1</maxVel>
+    <minDepth>0.003</minDepth>
     <sensor name="RFoot/FSR/FrontRight" type="contact">
       <always_on>1</always_on>
@@ -501,4 +542,11 @@
   </gazebo>
   <gazebo reference="LFsrRL_frame">
+    <mu1>0.5</mu1>
+    <mu2>0.5</mu2>
+    <selfCollide>false</selfCollide>
+    <turnGravityOff>false</turnGravityOff>
+    <fdir1>1 0 0</fdir1>
+    <maxVel>0.1</maxVel>
+    <minDepth>0.003</minDepth>
     <sensor name="LFoot/FSR/RearLeft" type="contact">
       <always_on>1</always_on>
@@ -512,4 +560,11 @@
   </gazebo>
   <gazebo reference="LFsrRR_frame">
+    <mu1>0.5</mu1>
+    <mu2>0.5</mu2>
+    <selfCollide>false</selfCollide>
+    <turnGravityOff>false</turnGravityOff>
+    <fdir1>1 0 0</fdir1>
+    <maxVel>0.1</maxVel>
+    <minDepth>0.003</minDepth>
     <sensor name="LFoot/FSR/RearRight" type="contact">
       <always_on>1</always_on>
@@ -523,4 +578,11 @@
   </gazebo>
   <gazebo reference="LFsrFL_frame">
+    <mu1>0.5</mu1>
+    <mu2>0.5</mu2>
+    <selfCollide>false</selfCollide>
+    <turnGravityOff>false</turnGravityOff>
+    <fdir1>1 0 0</fdir1>
+    <maxVel>0.1</maxVel>
+    <minDepth>0.003</minDepth>
     <sensor name="LFoot/FSR/FrontLeft" type="contact">
       <always_on>1</always_on>
@@ -534,4 +596,11 @@
   </gazebo>
   <gazebo reference="LFsrFR_frame">
+    <mu1>0.5</mu1>
+    <mu2>0.5</mu2>
+    <selfCollide>false</selfCollide>
+    <turnGravityOff>false</turnGravityOff>
+    <fdir1>1 0 0</fdir1>
+    <maxVel>0.1</maxVel>
+    <minDepth>0.003</minDepth>
     <sensor name="LFoot/FSR/FrontRight" type="contact">
       <always_on>1</always_on>
@@ -567,10 +636,10 @@
       <origin rpy="0 0 0" xyz="0 0 0"/>
     </visual>
-    <collision>
+    <!-- <collision>
       <geometry>
         <mesh filename="package://nao_meshes/meshes/V40/HeadYaw_0.10.stl" scale="0.1 0.1 0.1"/>
       </geometry>
       <origin rpy="0 0 0" xyz="0 0 0"/>
-    </collision>
+    </collision> -->
   </link>
   <joint name="HeadPitch" type="revolute">
@@ -598,8 +667,12 @@
     </visual>
     <collision>
-      <geometry>
+      <!-- <geometry>
         <mesh filename="package://nao_meshes/meshes/V40/HeadPitch_0.10.stl" scale="0.1 0.1 0.1"/>
       </geometry>
-      <origin rpy="0 0 0" xyz="0 0 0"/>
+      <origin rpy="0 0 0" xyz="0 0 0"/> -->
+      <origin xyz="0 0 0.058" rpy="1.57 0 0"/>
+      <geometry>
+          <cylinder radius="0.04" length="0.14"/>
+      </geometry>
     </collision>
   </link>
@@ -633,10 +706,10 @@
       <origin rpy="0 0 0" xyz="0 0 0"/>
     </visual>
-    <collision>
+    <!-- <collision>
       <geometry>
         <mesh filename="package://nao_meshes/meshes/V40/LHipYawPitch_0.10.stl" scale="0.1 0.1 0.1"/>
       </geometry>
       <origin rpy="0 0 0" xyz="0 0 0"/>
-    </collision>
+    </collision> -->
   </link>
   <joint name="LHipRoll" type="revolute">
@@ -663,10 +736,10 @@
       <origin rpy="0 0 0" xyz="0 0 0"/>
     </visual>
-    <collision>
+    <!-- <collision>
       <geometry>
         <mesh filename="package://nao_meshes/meshes/V40/LHipRoll_0.10.stl" scale="0.1 0.1 0.1"/>
       </geometry>
       <origin rpy="0 0 0" xyz="0 0 0"/>
-    </collision>
+    </collision> -->
   </link>
   <joint name="LHipPitch" type="revolute">
@@ -694,8 +767,12 @@
     </visual>
     <collision>
-      <geometry>
+      <!-- <geometry>
         <mesh filename="package://nao_meshes/meshes/V40/LHipPitch_0.10.stl" scale="0.1 0.1 0.1"/>
       </geometry>
-      <origin rpy="0 0 0" xyz="0 0 0"/>
+      <origin rpy="0 0 0" xyz="0 0 0"/> -->
+      <origin xyz="0 0 -0.05" rpy="0 0 0"/>
+      <geometry>
+          <cylinder radius="0.015" length="0.1"/>
+      </geometry>
     </collision>
   </link>
@@ -724,8 +801,12 @@
     </visual>
     <collision>
-      <geometry>
+      <!-- <geometry>
         <mesh filename="package://nao_meshes/meshes/V40/LKneePitch_0.10.stl" scale="0.1 0.1 0.1"/>
       </geometry>
-      <origin rpy="0 0 0" xyz="0 0 0"/>
+      <origin rpy="0 0 0" xyz="0 0 0"/> -->
+      <origin xyz="0 0 -0.05" rpy="0 0 0"/>
+      <geometry>
+          <cylinder radius="0.015" length="0.1"/>
+      </geometry>
     </collision>
   </link>
@@ -753,10 +834,10 @@
       <origin rpy="0 0 0" xyz="0 0 0"/>
     </visual>
-    <collision>
+    <!-- <collision>
       <geometry>
         <mesh filename="package://nao_meshes/meshes/V40/LAnklePitch_0.10.stl" scale="0.1 0.1 0.1"/>
       </geometry>
       <origin rpy="0 0 0" xyz="0 0 0"/>
-    </collision>
+    </collision> -->
   </link>
   <joint name="LAnkleRoll" type="revolute">
@@ -784,8 +865,12 @@
     </visual>
     <collision>
-      <geometry>
+      <!-- <geometry>
         <mesh filename="package://nao_meshes/meshes/V40/LAnkleRoll_0.10.stl" scale="0.1 0.1 0.1"/>
       </geometry>
-      <origin rpy="0 0 0" xyz="0 0 0"/>
+      <origin rpy="0 0 0" xyz="0 0 0"/> -->
+      <origin xyz="0.02 0.001 -0.038" rpy="0 0 0"/>
+      <geometry>
+          <box size="0.14 0.09 0.012"/>
+      </geometry>
     </collision>
   </link>
@@ -821,10 +906,10 @@
       <origin rpy="0 0 0" xyz="0 0 0"/>
     </visual>
-    <collision>
+    <!-- <collision>
       <geometry>
         <mesh filename="package://nao_meshes/meshes/V40/RHipYawPitch_0.10.stl" scale="0.1 0.1 0.1"/>
       </geometry>
       <origin rpy="0 0 0" xyz="0 0 0"/>
-    </collision>
+    </collision> -->
   </link>
   <joint name="RHipRoll" type="revolute">
@@ -851,10 +936,10 @@
       <origin rpy="0 0 0" xyz="0 0 0"/>
     </visual>
-    <collision>
+    <!-- <collision>
       <geometry>
         <mesh filename="package://nao_meshes/meshes/V40/RHipRoll_0.10.stl" scale="0.1 0.1 0.1"/>
       </geometry>
       <origin rpy="0 0 0" xyz="0 0 0"/>
-    </collision>
+    </collision> -->
   </link>
   <joint name="RHipPitch" type="revolute">
@@ -882,8 +967,12 @@
     </visual>
     <collision>
-      <geometry>
+      <!-- <geometry>
         <mesh filename="package://nao_meshes/meshes/V40/RHipPitch_0.10.stl" scale="0.1 0.1 0.1"/>
       </geometry>
-      <origin rpy="0 0 0" xyz="0 0 0"/>
+      <origin rpy="0 0 0" xyz="0 0 0"/> -->
+      <origin xyz="0 0 -0.05" rpy="0 0 0"/>
+      <geometry>
+          <cylinder radius="0.015" length="0.1"/>
+      </geometry>
     </collision>
   </link>
@@ -912,8 +1001,12 @@
     </visual>
     <collision>
-      <geometry>
+      <!-- <geometry>
         <mesh filename="package://nao_meshes/meshes/V40/RKneePitch_0.10.stl" scale="0.1 0.1 0.1"/>
       </geometry>
-      <origin rpy="0 0 0" xyz="0 0 0"/>
+      <origin rpy="0 0 0" xyz="0 0 0"/> -->
+      <origin xyz="0 0 -0.05" rpy="0 0 0"/>
+      <geometry>
+          <cylinder radius="0.015" length="0.1"/>
+      </geometry>
     </collision>
   </link>
@@ -941,10 +1034,10 @@
       <origin rpy="0 0 0" xyz="0 0 0"/>
     </visual>
-    <collision>
+    <!-- <collision>
       <geometry>
         <mesh filename="package://nao_meshes/meshes/V40/RAnklePitch_0.10.stl" scale="0.1 0.1 0.1"/>
       </geometry>
       <origin rpy="0 0 0" xyz="0 0 0"/>
-    </collision>
+    </collision> -->
   </link>
   <joint name="RAnkleRoll" type="revolute">
@@ -972,8 +1065,12 @@
     </visual>
     <collision>
-      <geometry>
+      <!-- <geometry>
         <mesh filename="package://nao_meshes/meshes/V40/RAnkleRoll_0.10.stl" scale="0.1 0.1 0.1"/>
       </geometry>
-      <origin rpy="0 0 0" xyz="0 0 0"/>
+      <origin rpy="0 0 0" xyz="0 0 0"/> -->
+      <origin xyz="0.02 -0.001 -0.038" rpy="0 0 0"/>
+      <geometry>
+          <box size="0.14 0.09 0.012"/>
+      </geometry>
     </collision>
   </link>
@@ -1005,8 +1102,13 @@
     </visual>
     <collision>
-      <geometry>
+      <!-- one cylinder spanning over HipOffsetZ and NeckOffsetZ -->
+      <origin xyz="0 0 0.02075" rpy="0 0 0"/>
+      <geometry>
+          <cylinder radius="0.015" length="0.2115"/>
+      </geometry>
+      <!-- <geometry>
         <mesh filename="package://nao_meshes/meshes/V40/Torso_0.10.stl" scale="0.1 0.1 0.1"/>
       </geometry>
-      <origin rpy="0 0 0" xyz="0 0 0"/>
+      <origin rpy="0 0 0" xyz="0 0 0"/> -->
     </collision>
   </link>
@@ -1034,10 +1136,10 @@
       <origin rpy="0 0 0" xyz="0 0 0"/>
     </visual>
-    <collision>
+    <!-- <collision>
       <geometry>
         <mesh filename="package://nao_meshes/meshes/V40/LShoulderPitch_0.10.stl" scale="0.1 0.1 0.1"/>
       </geometry>
       <origin rpy="0 0 0" xyz="0 0 0"/>
-    </collision>
+    </collision> -->
   </link>
   <joint name="LShoulderRoll" type="revolute">
@@ -1065,8 +1167,12 @@
     </visual>
     <collision>
-      <geometry>
+      <!-- <geometry>
         <mesh filename="package://nao_meshes/meshes/V40/LShoulderRoll_0.10.stl" scale="0.1 0.1 0.1"/>
       </geometry>
-      <origin rpy="0 0 0" xyz="0 0 0"/>
+      <origin rpy="0 0 0" xyz="0 0 0"/> -->
+      <origin xyz="0.045 0 0" rpy="1.57079632679 0 1.57079632679"/>
+      <geometry>
+          <cylinder radius="0.015" length="0.09"/>
+      </geometry>
     </collision>
   </link>
@@ -1113,8 +1219,12 @@
     </visual>
     <collision>
-      <geometry>
+      <!-- <geometry>
         <mesh filename="package://nao_meshes/meshes/V40/LElbowRoll_0.10.stl" scale="0.1 0.1 0.1"/>
       </geometry>
-      <origin rpy="0 0 0" xyz="0 0 0"/>
+      <origin rpy="0 0 0" xyz="0 0 0"/> -->
+      <origin xyz="0.025325 0 0" rpy="1.57079632679 0 1.57079632679"/>
+      <geometry>
+          <cylinder radius="0.015" length="0.05065"/>
+      </geometry>
     </collision>
   </link>
@@ -1143,8 +1253,12 @@
     </visual>
     <collision>
-      <geometry>
+      <!-- <geometry>
         <mesh filename="package://nao_meshes/meshes/V40/LWristYaw_0.10.stl" scale="0.1 0.1 0.1"/>
       </geometry>
-      <origin rpy="0 0 0" xyz="0 0 0"/>
+      <origin rpy="0 0 0" xyz="0 0 0"/> -->
+      <origin xyz="0.029 0 0" rpy="1.57079632679 0 1.57079632679"/>
+      <geometry>
+          <cylinder radius="0.015" length="0.058"/>
+      </geometry>
     </collision>
   </link>
@@ -1189,10 +1303,10 @@
       <origin rpy="0 0 0" xyz="0 0 0"/>
     </visual>
-    <collision>
+    <!-- <collision>
       <geometry>
         <mesh filename="package://nao_meshes/meshes/V40/RShoulderPitch_0.10.stl" scale="0.1 0.1 0.1"/>
       </geometry>
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