Commit message: Returned to full collision meshes, small fixes in plugin code

File: gazebo_naoqi_control/models/nao.xacro (robot description, xacro)
@@ -385,10 +385,10 @@
     </sensor>
   </gazebo>
-  <!-- <gazebo reference="LSonar_frame">
+  <gazebo reference="LSonar_frame">
     <sensor name="Sonar/Left" type="ray">
       <pose>0 0 0 0 0 0</pose>
       <always_on>1</always_on>
       <update_rate>20</update_rate>
-      <visualize>true</visualize>
+      <visualize>false</visualize>
       <ray>
         <scan>
@@ -409,6 +409,11 @@
           <min>0.025</min>
           <max>2.55</max>
-          <resolution>0.01</resolution>
+          <resolution>1</resolution>
         </range>
+        <noise>
+          <type>gaussian</type>
+          <mean>0.0</mean>
+          <stddev>0.05</stddev>
+        </noise>
       </ray>
     </sensor>
@@ -419,5 +424,5 @@
       <always_on>1</always_on>
       <update_rate>20</update_rate>
-      <visualize>true</visualize>
+      <visualize>false</visualize>
       <ray>
         <scan>
@@ -438,33 +443,12 @@
           <min>0.025</min>
           <max>2.55</max>
-          <resolution>0.01</resolution>
+          <resolution>1</resolution>
         </range>
+        <noise>
+          <type>gaussian</type>
+          <mean>0.0</mean>
+          <stddev>0.05</stddev>
+        </noise>
       </ray>
-    </sensor>
-  </gazebo> -->
-  <gazebo reference="LSonar_frame">
-    <sensor name="Sonar/Left" type="sonar">
-      <always_on>1</always_on>
-      <update_rate>20</update_rate>
-      <visualize>false</visualize>
-      <sonar>
-        <min>0.025</min>
-        <max>2.55</max>
-        <!-- NEEDS TWEAKING -->
-        <radius>0.25</radius>
-      </sonar>
-    </sensor>
-  </gazebo>
-  <gazebo reference="RSonar_frame">
-    <sensor name="Sonar/Right" type="sonar">
-      <always_on>1</always_on>
-      <update_rate>20</update_rate>
-      <visualize>false</visualize>
-      <sonar>
-        <min>0.025</min>
-        <max>2.55</max>
-        <!-- NEEDS TWEAKING -->
-        <radius>0.25</radius>
-      </sonar>
     </sensor>
   </gazebo>
@@ -636,10 +620,10 @@
       <origin rpy="0 0 0" xyz="0 0 0"/>
     </visual>
-    <!-- <collision>
+    <collision>
       <geometry>
         <mesh filename="package://nao_meshes/meshes/V40/HeadYaw_0.10.stl" scale="0.1 0.1 0.1"/>
       </geometry>
       <origin rpy="0 0 0" xyz="0 0 0"/>
-    </collision> -->
+    </collision>
   </link>
   <joint name="HeadPitch" type="revolute">
@@ -667,12 +651,12 @@
     </visual>
     <collision>
-      <!-- <geometry>
+      <geometry>
         <mesh filename="package://nao_meshes/meshes/V40/HeadPitch_0.10.stl" scale="0.1 0.1 0.1"/>
       </geometry>
-      <origin rpy="0 0 0" xyz="0 0 0"/> -->
-      <origin xyz="0 0 0.058" rpy="1.57 0 0"/>
+      <origin rpy="0 0 0" xyz="0 0 0"/>
+      <!-- <origin xyz="0 0 0.058" rpy="1.57 0 0"/>
       <geometry>
           <cylinder radius="0.04" length="0.14"/>
-      </geometry>
+      </geometry> -->
     </collision>
   </link>
@@ -706,10 +690,10 @@
       <origin rpy="0 0 0" xyz="0 0 0"/>
     </visual>
-    <!-- <collision>
+    <collision>
       <geometry>
         <mesh filename="package://nao_meshes/meshes/V40/LHipYawPitch_0.10.stl" scale="0.1 0.1 0.1"/>
       </geometry>
       <origin rpy="0 0 0" xyz="0 0 0"/>
-    </collision> -->
+    </collision>
   </link>
   <joint name="LHipRoll" type="revolute">
@@ -736,10 +720,10 @@
       <origin rpy="0 0 0" xyz="0 0 0"/>
     </visual>
-    <!-- <collision>
+    <collision>
       <geometry>
         <mesh filename="package://nao_meshes/meshes/V40/LHipRoll_0.10.stl" scale="0.1 0.1 0.1"/>
       </geometry>
       <origin rpy="0 0 0" xyz="0 0 0"/>
-    </collision> -->
+    </collision>
   </link>
   <joint name="LHipPitch" type="revolute">
@@ -767,12 +751,12 @@
     </visual>
     <collision>
-      <!-- <geometry>
+      <geometry>
         <mesh filename="package://nao_meshes/meshes/V40/LHipPitch_0.10.stl" scale="0.1 0.1 0.1"/>
       </geometry>
-      <origin rpy="0 0 0" xyz="0 0 0"/> -->
-      <origin xyz="0 0 -0.05" rpy="0 0 0"/>
+      <origin rpy="0 0 0" xyz="0 0 0"/>
+      <!-- <origin xyz="0 0 -0.05" rpy="0 0 0"/>
       <geometry>
           <cylinder radius="0.015" length="0.1"/>
-      </geometry>
+      </geometry> -->
     </collision>
   </link>
@@ -801,12 +785,12 @@
     </visual>
     <collision>
-      <!-- <geometry>
+      <geometry>
         <mesh filename="package://nao_meshes/meshes/V40/LKneePitch_0.10.stl" scale="0.1 0.1 0.1"/>
       </geometry>
-      <origin rpy="0 0 0" xyz="0 0 0"/> -->
-      <origin xyz="0 0 -0.05" rpy="0 0 0"/>
+      <origin rpy="0 0 0" xyz="0 0 0"/>
+      <!-- <origin xyz="0 0 -0.05" rpy="0 0 0"/>
       <geometry>
           <cylinder radius="0.015" length="0.1"/>
-      </geometry>
+      </geometry> -->
     </collision>
   </link>
@@ -834,10 +818,10 @@
       <origin rpy="0 0 0" xyz="0 0 0"/>
     </visual>
-    <!-- <collision>
+    <collision>
       <geometry>
         <mesh filename="package://nao_meshes/meshes/V40/LAnklePitch_0.10.stl" scale="0.1 0.1 0.1"/>
       </geometry>
       <origin rpy="0 0 0" xyz="0 0 0"/>
-    </collision> -->
+    </collision>
   </link>
   <joint name="LAnkleRoll" type="revolute">
@@ -865,12 +849,12 @@
     </visual>
     <collision>
-      <!-- <geometry>
+      <geometry>
         <mesh filename="package://nao_meshes/meshes/V40/LAnkleRoll_0.10.stl" scale="0.1 0.1 0.1"/>
       </geometry>
-      <origin rpy="0 0 0" xyz="0 0 0"/> -->
-      <origin xyz="0.02 0.001 -0.038" rpy="0 0 0"/>
+      <origin rpy="0 0 0" xyz="0 0 0"/>
+      <!-- <origin xyz="0.02 0.001 -0.038" rpy="0 0 0"/>
       <geometry>
           <box size="0.14 0.09 0.012"/>
-      </geometry>
+      </geometry> -->
     </collision>
   </link>
@@ -906,10 +890,10 @@
       <origin rpy="0 0 0" xyz="0 0 0"/>
     </visual>
-    <!-- <collision>
+    <collision>
       <geometry>
         <mesh filename="package://nao_meshes/meshes/V40/RHipYawPitch_0.10.stl" scale="0.1 0.1 0.1"/>
       </geometry>
       <origin rpy="0 0 0" xyz="0 0 0"/>
-    </collision> -->
+    </collision>
   </link>
   <joint name="RHipRoll" type="revolute">
@@ -936,10 +920,10 @@
       <origin rpy="0 0 0" xyz="0 0 0"/>
     </visual>
-    <!-- <collision>
+    <collision>
       <geometry>
         <mesh filename="package://nao_meshes/meshes/V40/RHipRoll_0.10.stl" scale="0.1 0.1 0.1"/>
       </geometry>
       <origin rpy="0 0 0" xyz="0 0 0"/>
-    </collision> -->
+    </collision>
   </link>
   <joint name="RHipPitch" type="revolute">
@@ -967,12 +951,12 @@
     </visual>
     <collision>
-      <!-- <geometry>
+      <geometry>
         <mesh filename="package://nao_meshes/meshes/V40/RHipPitch_0.10.stl" scale="0.1 0.1 0.1"/>
       </geometry>
-      <origin rpy="0 0 0" xyz="0 0 0"/> -->
-      <origin xyz="0 0 -0.05" rpy="0 0 0"/>
+      <origin rpy="0 0 0" xyz="0 0 0"/>
+      <!-- <origin xyz="0 0 -0.05" rpy="0 0 0"/>
       <geometry>
           <cylinder radius="0.015" length="0.1"/>
-      </geometry>
+      </geometry> -->
     </collision>
   </link>
@@ -1001,12 +985,12 @@
     </visual>
     <collision>
-      <!-- <geometry>
+      <geometry>
         <mesh filename="package://nao_meshes/meshes/V40/RKneePitch_0.10.stl" scale="0.1 0.1 0.1"/>
       </geometry>
-      <origin rpy="0 0 0" xyz="0 0 0"/> -->
-      <origin xyz="0 0 -0.05" rpy="0 0 0"/>
+      <origin rpy="0 0 0" xyz="0 0 0"/>
+      <!-- <origin xyz="0 0 -0.05" rpy="0 0 0"/>
       <geometry>
           <cylinder radius="0.015" length="0.1"/>
-      </geometry>
+      </geometry> -->
     </collision>
   </link>
@@ -1034,10 +1018,10 @@
       <origin rpy="0 0 0" xyz="0 0 0"/>
     </visual>
-    <!-- <collision>
+    <collision>
       <geometry>
         <mesh filename="package://nao_meshes/meshes/V40/RAnklePitch_0.10.stl" scale="0.1 0.1 0.1"/>
       </geometry>
       <origin rpy="0 0 0" xyz="0 0 0"/>
-    </collision> -->
+    </collision>
   </link>
   <joint name="RAnkleRoll" type="revolute">
@@ -1065,12 +1049,12 @@
     </visual>
     <collision>
-      <!-- <geometry>
+      <geometry>
         <mesh filename="package://nao_meshes/meshes/V40/RAnkleRoll_0.10.stl" scale="0.1 0.1 0.1"/>
       </geometry>
-      <origin rpy="0 0 0" xyz="0 0 0"/> -->
-      <origin xyz="0.02 -0.001 -0.038" rpy="0 0 0"/>
+      <origin rpy="0 0 0" xyz="0 0 0"/>
+      <!-- <origin xyz="0.02 -0.001 -0.038" rpy="0 0 0"/>
       <geometry>
           <box size="0.14 0.09 0.012"/>
-      </geometry>
+      </geometry> -->
     </collision>
   </link>
@@ -1102,13 +1086,12 @@
     </visual>
     <collision>
-      <!-- one cylinder spanning over HipOffsetZ and NeckOffsetZ -->
-      <origin xyz="0 0 0.02075" rpy="0 0 0"/>
+      <!-- <origin xyz="0 0 0.02075" rpy="0 0 0"/>
       <geometry>
           <cylinder radius="0.015" length="0.2115"/>
-      </geometry>
-      <!-- <geometry>
+      </geometry> -->
+      <geometry>
         <mesh filename="package://nao_meshes/meshes/V40/Torso_0.10.stl" scale="0.1 0.1 0.1"/>
       </geometry>
-      <origin rpy="0 0 0" xyz="0 0 0"/> -->
+      <origin rpy="0 0 0" xyz="0 0 0"/>
     </collision>
   </link>
@@ -1136,10 +1119,10 @@
       <origin rpy="0 0 0" xyz="0 0 0"/>
     </visual>
-    <!-- <collision>
+    <collision>
       <geometry>
         <mesh filename="package://nao_meshes/meshes/V40/LShoulderPitch_0.10.stl" scale="0.1 0.1 0.1"/>
       </geometry>
       <origin rpy="0 0 0" xyz="0 0 0"/>
-    </collision> -->
+    </collision>
   </link>
   <joint name="LShoulderRoll" type="revolute">
@@ -1167,12 +1150,12 @@
     </visual>
     <collision>
-      <!-- <geometry>
+      <geometry>
         <mesh filename="package://nao_meshes/meshes/V40/LShoulderRoll_0.10.stl" scale="0.1 0.1 0.1"/>
       </geometry>
-      <origin rpy="0 0 0" xyz="0 0 0"/> -->
-      <origin xyz="0.045 0 0" rpy="1.57079632679 0 1.57079632679"/>
+      <origin rpy="0 0 0" xyz="0 0 0"/>
+      <!-- <origin xyz="0.045 0 0" rpy="1.57079632679 0 1.57079632679"/>
       <geometry>
           <cylinder radius="0.015" length="0.09"/>
-      </geometry>
+      </geometry> -->
     </collision>
   </link>
@@ -1219,12 +1202,12 @@
     </visual>
     <collision>
-      <!-- <geometry>
+      <geometry>
         <mesh filename="package://nao_meshes/meshes/V40/LElbowRoll_0.10.stl" scale="0.1 0.1 0.1"/>
       </geometry>
-      <origin rpy="0 0 0" xyz="0 0 0"/> -->
-      <origin xyz="0.025325 0 0" rpy="1.57079632679 0 1.57079632679"/>
+      <origin rpy="0 0 0" xyz="0 0 0"/>
+      <!-- <origin xyz="0.025325 0 0" rpy="1.57079632679 0 1.57079632679"/>
       <geometry>
           <cylinder radius="0.015" length="0.05065"/>
-      </geometry>
+      </geometry> -->
     </collision>
   </link>
@@ -1253,12 +1236,12 @@
     </visual>
     <collision>
-      <!-- <geometry>
+      <geometry>
         <mesh filename="package://nao_meshes/meshes/V40/LWristYaw_0.10.stl" scale="0.1 0.1 0.1"/>
       </geometry>
-      <origin rpy="0 0 0" xyz="0 0 0"/> -->
-      <origin xyz="0.029 0 0" rpy="1.57079632679 0 1.57079632679"/>
+      <origin rpy="0 0 0" xyz="0 0 0"/>
+      <!-- <origin xyz="0.029 0 0" rpy="1.57079632679 0 1.57079632679"/>
       <geometry>
           <cylinder radius="0.015" length="0.058"/>
-      </geometry>
+      </geometry> -->
     </collision>
   </link>
@@ -1303,10 +1286,10 @@
       <origin rpy="0 0 0" xyz="0 0 0"/>
     </visual>
-    <!-- <collision>
+    <collision>
       <geometry>
         <mesh filename="package://nao_meshes/meshes/V40/RShoulderPitch_0.10.stl" scale="0.1 0.1 0.1"/>
       </geometry>
       <origin rpy="0 0 0" xyz="0 0 0"/>
-    </collision> -->
+    </collision>
   </link>
   <joint name="RShoulderRoll" type="revolute">
@@ -1334,12 +1317,12 @@
     </visual>
     <collision>
-      <!-- <geometry>
+      <geometry>
         <mesh filename="package://nao_meshes/meshes/V40/RShoulderRoll_0.10.stl" scale="0.1 0.1 0.1"/>
       </geometry>
-      <origin rpy="0 0 0" xyz="0 0 0"/> -->
-      <origin xyz="0.045 0 0" rpy="1.57079632679 0 1.57079632679"/>
+      <origin rpy="0 0 0" xyz="0 0 0"/>
+      <!-- <origin xyz="0.045 0 0" rpy="1.57079632679 0 1.57079632679"/>
       <geometry>
           <cylinder radius="0.015" length="0.09"/>
-      </geometry>
+      </geometry> -->
     </collision>
   </link>
@@ -1386,12 +1369,12 @@
     </visual>
     <collision>
-      <!-- <geometry>
+      <geometry>
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
Commit message: Changed collisions of feet back to simple rectangles

File: gazebo_naoqi_control/models/nao.xacro (robot description, xacro)
@@ -849,12 +849,12 @@
     </visual>
     <collision>
-      <geometry>
+      <!-- <geometry>
         <mesh filename="package://nao_meshes/meshes/V40/LAnkleRoll_0.10.stl" scale="0.1 0.1 0.1"/>
       </geometry>
-      <origin rpy="0 0 0" xyz="0 0 0"/>
-      <!-- <origin xyz="0.02 0.001 -0.038" rpy="0 0 0"/>
+      <origin rpy="0 0 0" xyz="0 0 0"/> -->
+      <origin xyz="0.02 0.001 -0.038" rpy="0 0 0"/>
       <geometry>
           <box size="0.14 0.09 0.012"/>
-      </geometry> -->
+      </geometry>
     </collision>
   </link>
@@ -1049,12 +1049,12 @@
     </visual>
     <collision>
-      <geometry>
+      <!-- <geometry>
         <mesh filename="package://nao_meshes/meshes/V40/RAnkleRoll_0.10.stl" scale="0.1 0.1 0.1"/>
       </geometry>
-      <origin rpy="0 0 0" xyz="0 0 0"/>
-      <!-- <origin xyz="0.02 -0.001 -0.038" rpy="0 0 0"/>
+      <origin rpy="0 0 0" xyz="0 0 0"/> -->
+      <origin xyz="0.02 -0.001 -0.038" rpy="0 0 0"/>
       <geometry>
           <box size="0.14 0.09 0.012"/>
-      </geometry> -->
+      </geometry>
     </collision>
   </link>
